Commit message: Simulate the dome servos and mirror the real servo device
The <astromech:servo> joints had no actuation in Gazebo, so they swung
freely while /joint_states reported zero. The sim now drives them
through the same contract as the dome servo device (r2_domeplayer):
/dome/joint_command in, /dome/joint_states out.

- Dome panels: a per-joint gz-sim JointPositionController in velocity
  mode moves each panel at a constant speed to its target, like the
  real servos. Joints and speeds are in config/dome_servos.yaml
  (16 rad/s, ~100 ms full travel); panels spawn closed.
- Body panels and utility arms: held closed by the servo_pos
  JointGroupPositionController (joint list in sim_controllers.yaml).
- New servo_sim node:
  - mirrors /dome/joint_states into Gazebo (per-joint cmd_pos topics
    bridged by servo_bridge, or servo_pos), forwarding as states arrive;
  - with servo_device:=sim emulates the device for the dome servos in
    /robot_description: name with or without _joint, clamp to the URDF
    limits, refuse unknown joints, publish the commanded target at
    10 Hz and on each command;
  - mutes any joint a real device on the network has reported within
    the last second (claim_timeout), so a partially configured device
    drives its servos and the sim fills in the rest. Its own messages
    carry header.frame_id "servo_sim".
- servo_device:=real disables emulation so only the real device drives
  the panels (hardware in the loop).
- README: servo setup, per-joint speeds and the HIL options.

Requires r2_bringup with /dome/joint_states in joint_state_publisher's
source_list.

Co-Authored-By: Claude Opus 5.5 <noreply@anthropic.com>

File: urdf/gz_ros2_control.xacro (robot description, xacro)
@@ -2,4 +2,41 @@
 <robot xmlns:xacro="http://www.ros.org/wiki/xacro">
     <xacro:if value="$(arg sim_mode)">
+        <!-- Body panels and utility arms come from the servo_pos controller's joint list,
+             so they're defined once -->
+        <xacro:property name="servo_joints"
+                        value="${xacro.load_yaml('$(find r2_sim)/config/sim_controllers.yaml')['servo_pos']['ros__parameters']['joints']}" />
+        <!-- Position-held servo joint, starting closed (0 is every servo's lower limit) -->
+        <xacro:macro name="servo_position_joints" params="joints">
+            <xacro:if value="${len(joints) > 0}">
+                <joint name="${joints[0]}">
+                    <command_interface name="position" />
+                    <state_interface name="position">
+                        <param name="initial_value">0.0</param>
+                    </state_interface>
+                    <state_interface name="velocity" />
+                </joint>
+                <xacro:servo_position_joints joints="${joints[1:]}" />
+            </xacro:if>
+        </xacro:macro>
+        <!-- Dome panels: Gazebo drives each one like a servo, at a constant speed to its target.
+             With use_velocity_commands, cmd_max is that speed in rad/s. Commands arrive on
+             /servo/<joint>/cmd_pos (bridged from ROS in launch_sim.launch.py). -->
+        <xacro:property name="dome_servos" value="${xacro.load_yaml('$(find r2_sim)/config/dome_servos.yaml')}" />
+        <xacro:macro name="dome_servo_controllers" params="joints">
+            <xacro:if value="${len(joints) > 0}">
+                <xacro:property name="velocity" value="${dome_servos[joints[0]]['velocity']}" />
+                <gazebo>
+                    <plugin name="gz::sim::systems::JointPositionController" filename="gz-sim-joint-position-controller-system">
+                        <joint_name>${joints[0]}</joint_name>
+                        <topic>/servo/${joints[0]}/cmd_pos</topic>
+                        <use_velocity_commands>true</use_velocity_commands>
+                        <cmd_max>${velocity}</cmd_max>
+                        <cmd_min>${-velocity}</cmd_min>
+                        <initial_position>0.0</initial_position>
+                    </plugin>
+                </gazebo>
+                <xacro:dome_servo_controllers joints="${joints[1:]}" />
+            </xacro:if>
+        </xacro:macro>
         <ros2_control name="GazeboSystem" type="system">
             <hardware>
@@ -60,5 +97,7 @@
                 <state_interface name="position" />
             </joint>
+            <xacro:servo_position_joints joints="${servo_joints}" />
         </ros2_control>
+        <xacro:dome_servo_controllers joints="${list(dome_servos.keys())}" />
         <gazebo>
             <plugin name="gz_ros2_control::GazeboSimROS2ControlPlugin" filename="libgz_ros2_control-system.so">
